Commit message: Need to sort out thruster issues and figure out why vehicle is sinking.

File: urdf/videoray_pro4.xacro (robot description, xacro)
@@ -10,5 +10,6 @@
   <xacro:property name="mass" value="6.123497"/>
   <!-- Volume taken from mesh in Blender. Should be verified in Solidworks or similar to ensure it uses the face of the mesh to calculate volume. -->
-  <xacro:property name="volume" value="0.0031093918"/>
+  <!-- <xacro:property name="volume" value="0.0031093918"/> -->
+  <xacro:property name="volume" value="3.1093918"/>
   <!-- Center of gravity. Assumption, should be checked.-->
   <xacro:property name="cog" value="0 0 0"/>
@@ -39,5 +40,5 @@
        </inertial>
        <visual>
-        <origin xyz="0 0 0" rpy="0 0 0"/>
+        <origin xyz="0 0 0" rpy="0 0 -1.57"/>
         <geometry>
           <mesh filename="${visual_mesh_file}" scale="1 1 1" />
@@ -45,5 +46,5 @@
       </visual>
       <collision>
-        <origin xyz="0 0 0" rpy="0 0 0"/>
+        <origin xyz="0 0 0" rpy="0 0 -1.57"/>
         <geometry>
           <mesh filename="${collision_mesh_file}" scale="1 1 1" />

File: urdf/videoray_pro4_sensors.xacro (robot description, xacro)
@@ -13,11 +13,11 @@
   </gazebo>
   <!-- DVL  -->
-  <xacro:default_dvl namespace="${namespace}" parent_link="${namespace}/base_link">
+  <!-- <xacro:default_dvl namespace="${namespace}" parent_link="${namespace}/base_link">
     <origin xyz="0 0 0" rpy="0 0 0"/>
-  </xacro:default_dvl>
+  </xacro:default_dvl> -->
   <!-- RPT  -->
-  <xacro:default_rpt namespace="${namespace}" parent_link="${namespace}/base_link">
+  <!-- <xacro:default_rpt namespace="${namespace}" parent_link="${namespace}/base_link">
     <origin xyz="0 0 0" rpy="0 0 0"/>
-  </xacro:default_rpt>
+  </xacro:default_rpt> -->
   <!-- Pressure  -->
   <xacro:default_pressure namespace="${namespace}" parent_link="${namespace}/base_link">

File: urdf/videoray_pro4_thruster.xacro (robot description, xacro)
@@ -27,42 +27,43 @@
     </link>
     <!-- Joint between thruster link and vehicle base link -->
-        <joint name="${robot_namespace}/thruster_${thruster_id}_joint" type="continuous">
-          <xacro:insert_block name="origin" />
-          <axis xyz="1 0 0" />
-          <parent link="${robot_namespace}/base_link" />
-          <child link="${robot_namespace}/thruster_${thruster_id}" />
-        </joint>
-    <gazebo>
-    	<!-- Thruster ROS plugin -->
-    	<plugin name="${robot_namespace}_${thruster_id}_thruster_model" filename="libthruster_ros_plugin.so">
-    		<!-- Name of the thruster link -->
-    		<linkName>${robot_namespace}/thruster_${thruster_id}</linkName>
-    		<!-- Name of the joint between thruster and vehicle base link -->
-    		<jointName>${robot_namespace}/thruster_${thruster_id}_joint</jointName>
-    		<!-- Thruster force output topic name -->
-    		<thrustTopic>${robot_namespace}/thrusters/${thruster_id}/thrust</thrustTopic>
-    		<!-- Thruster commmand input topic name -->
-    		<inputTopic>${robot_namespace}/thrusters/${thruster_id}/input</inputTopic>
-    		<!-- Gain of the input command signal -->
-    		<gain>1</gain>
-    		<!-- Maximum allowed input value for the input signal for thruster unit -->
-    		<clampMax>2</clampMax>
-    		<!-- Minimum allowed value for the input signal for thruster unit -->
-    		<clampMin>0</clampMin>
-    		<thrust_efficiency>1</thrust_efficiency>
-    		<propeller_efficiency>1</propeller_efficiency>
-    		<!-- Simple zero-order model -->
-    		<dynamics>
-    			<type>ZeroOrder</type>
-    		</dynamics>
-    		<conversion>
-    			<type>Basic</type>
-    			<rotorConstant>10</rotorConstant>
-    		</conversion>
-    	</plugin>
-    </gazebo>
-    <gazebo reference="${robot_namespace}/thruster_${thruster_id}">
-    	<selfCollide>false</selfCollide>
-    </gazebo>
+    <joint name="${robot_namespace}/thruster_${thruster_id}_joint" type="continuous">
+      <xacro:insert_block name="origin" />
+      <axis xyz="0 0 1" />
+      <parent link="${robot_namespace}/base_link" />
+      <child link="${robot_namespace}/thruster_${thruster_id}" />
+  </joint>
+  <gazebo>
+   <!-- Thruster ROS plugin -->
+   <plugin name="${robot_namespace}_${thruster_id}_thruster_model" filename="libthruster_ros_plugin.so">
+      <!-- Name of the thruster link -->
+      <linkName>${robot_namespace}/thruster_${thruster_id}</linkName>
+      <!-- Name of the joint between thruster and vehicle base link -->
+      <jointName>${robot_namespace}/thruster_${thruster_id}_joint</jointName>
+      <thrusterID>${thruster_id}</thrusterID>
+      <!-- Thruster force output topic name -->
+      <thrustTopic>${robot_namespace}/thrusters/${thruster_id}/thrust</thrustTopic>
+      <!-- Thruster commmand input topic name -->
+      <inputTopic>${robot_namespace}/thrusters/${thruster_id}/input</inputTopic>
+      <!-- Gain of the input command signal -->
+      <gain>1</gain>
+      <!-- Maximum allowed input value for the input signal for thruster unit -->
+      <clampMax>2</clampMax>
+      <!-- Minimum allowed value for the input signal for thruster unit -->
+      <clampMin>0</clampMin>
+      <thrust_efficiency>1</thrust_efficiency>
+      <propeller_efficiency>1</propeller_efficiency>
+      <dynamics>
+          <type>FirstOrder</type>
+          <timeConstant>0.05</timeConstant>
+      </dynamics>
+      <conversion>
+         <type>Basic</type>
+         <rotorConstant>0.00031</rotorConstant>
+     </conversion>
+ </plugin>
+</gazebo>
+<gazebo reference="${robot_namespace}/thruster_${thruster_id}">
+   <selfCollide>false</selfCollide>
+</gazebo>
 </xacro:macro>
 </robot>

Commit message: Added thruster manager and associated config/launch files.

File: urdf/videoray_pro4.xacro (robot description, xacro)
@@ -9,13 +9,12 @@
   <!-- Vehicle's parameters -->
   <xacro:property name="mass" value="6.123497"/>
-  <!-- Volume taken from mesh in Blender. Should be verified in Solidworks or similar to ensure it uses the face of the mesh to calculate volume. -->
-  <!-- <xacro:property name="volume" value="0.0031093918"/> -->
-  <xacro:property name="volume" value="3.1093918"/>
+  <!-- <xacro:property name="mass" value="0.123497"/> -->
+  <xacro:property name="volume" value="0.051093918"/>
   <!-- Center of gravity. Assumption, should be checked.-->
   <xacro:property name="cog" value="0 0 0"/>
   <!-- Center of buoyancy -->
-  <xacro:property name="cob" value="0 0 0.15"/>
+  <xacro:property name="cob" value="0 0 0.25"/>
   <!-- Fluid density, assuming fresh water right now. For salt water, use 1028 or so. -->
-  <xacro:property name="rho" value="1000"/>
+  <xacro:property name="rho" value="1028"/>
   <!-- Describing the dimensions of the vehicle's bounding box -->
   <xacro:property name="length" value="0.375"/>
@@ -35,7 +34,7 @@
         <mass value="${mass}" />
         <origin xyz="${cog}" rpy="0 0 0"/>
-        <inertia ixx="0" ixy="0" ixz="0"
-         iyy="0" iyz="0"
-         izz="0" />
+        <inertia ixx="0.16319" ixy="0" ixz="0"
+         iyy="0.23313" iyz="0"
+         izz="0.27451" />
        </inertial>
        <visual>
@@ -59,4 +58,5 @@
   <xacro:dummy_link name="${namespace}/ned_link" />
   <joint name="ned_joint" type="revolute">
+  <!-- <joint name="ned_joint" type="fixed"> -->
     <!-- This is revolute and not static since gazebo would remove ned_link -->
     <origin xyz="0 0 0" rpy="${pi} 0 0"/>
@@ -79,5 +79,5 @@
         <link name="${namespace}/base_link">
           <!-- This flag will make the link neutrally buoyant -->
-          <neutrally_buoyant>0</neutrally_buoyant>
+          <neutrally_buoyant>1</neutrally_buoyant>
           <!-- Link's volume -->
           <volume>${volume}</volume>
@@ -85,8 +85,13 @@
           volume when close to the surface.
           This is a workaround the invalid bounding box given by Gazebo-->
-          <box>
+          <!-- <box>
             <width>${width}</width>
             <length>${length}</length>
             <height>${height}</height>
+          </box> -->
+          <box>
+            <width>1.5</width>
+            <length>2.6</length>
+            <height>1.6</height>
           </box>
           <!-- Center of buoyancy -->
@@ -94,4 +99,5 @@
           <hydrodynamic_model>
             <type>fossen</type>
+            <!-- Added mass: see p.28 in Berg2012 -->
             <added_mass>
               0 0 0 0 0 0
@@ -102,10 +108,18 @@
               0 0 0 0 0 0
             </added_mass>
+            <!-- Linear damping: see p.31 in Berg2012 -->
             <linear_damping>
-              0 0 0 0 0 0
+              -7.82 -6.48 -72.4 -26.8 -30.77 -10
             </linear_damping>
+            <!-- Non-linear damping: see p.30 in Berg2012 -->
+            <quadratic_damping>
+              -78.22 -92.53 -181.01 -67 -77.44 -52.27
+            </quadratic_damping>
           </hydrodynamic_model>
         </link>
       </plugin>
+    </gazebo>
+    <gazebo reference="${namespace}/base_link">
+      <material>Gazebo/Orange</material>
     </gazebo>
     <!-- Include the thruster modules -->
